File: hardware/design/shot-detector/shot-detector.kicad_pcb (KiCad board)
At the start: 2 copper layers, 21 x 18 mm, 11 parts, among them J1 Conn_01x05, J2 Conn_01x05, J3 Conn_01x05, U1 LM393

Commit message: First pass of PCB layout.
Parts:
- removed D3: LED, LED_SMD:LED_1206_3216Metric
- removed R3: 1k, Resistor_SMD:R_1206_3216Metric
- C1, J2, R2: moved to B.Cu
- moved J2 7.98 mm to (63.1, 90.1), turned to 180 degrees
- moved R1 0.63 mm to (59.0, 81.7)
- moved R2 0.15 mm to (55.6, 85.6), turned to 90 degrees
- moved C1 0.12 mm to (53.0, 85.6)
Routing:
- net /pizo_conditioned: track 0.00 -> 25.1 mm, vias 0 -> 1
- net +5V: track 0.00 -> 17.5 mm, vias 0 -> 2
- net /output: track 0.33 -> 12.3 mm, vias 0 -> 1
- net /pizo_in: track 0.00 -> 7.57 mm, vias 0 -> 2
- net GND: track 0.00 -> 4.17 mm, vias 0 -> 1
- added copper zone on F.Cu, net GND
- removed copper zone on B.Cu, net (none)
Other:
- board size 21 x 18 mm -> 21 x 13.5 mm

Commit message: V1 of PCB ordered.
Other:
- board text added: "v1"
Changed lines of the file:
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@@
 			(outputformat 1)
 			(mirror no)
-			(drillshape 1)
+			(drillshape 0)
 			(scaleselection 1)
 			(outputdirectory "")
@@
 			(type solid)
 		)
-		(layer "Dwgs.User")
+		(layer "Cmts.User")
 	)
 	(gr_line
@@
 		(layer "Edge.Cuts")
 	)
+	(gr_text "v1"
+		(at 54.55 80.45 0)
+		(layer "B.SilkS")
+		(effects
+			(font
+				(size 1.5 1.5)
+				(thickness 0.3)
+				(bold yes)
+			)
+			(justify left bottom mirror)
+		)
+	)
 	(via
